File: pts.kicad_sch (KiCad schematic)
At the start: 7 parts, among them U8 OPA357

Commit message: fixed resistor values
Changed lines of the file:
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@@
   (symbol (lib_id "Device:R_Small_US") (at 81.28 54.61 90) (unit 1)
     (in_bom yes) (on_board yes) (dnp no)
-    (property "Reference" "R10" (at 80.01 52.07 0)
+    (property "Reference" "R10" (at 83.185 50.165 90)
       (effects (font (size 1.27 1.27)) (justify left))
     )
-    (property "Value" "1K" (at 82.55 52.07 0)
+    (property "Value" "1K" (at 82.55 52.07 90)
       (effects (font (size 1.27 1.27)) (justify left))
     )

Commit message: added full schematic and outdated pcb
Parts:
- C30: symbol Device:C_Small -> UCIRP-KiCAD-Lib:C_Small
- D3: symbol Device:D_Zener_Small -> UCIRP-KiCAD-Lib:D_Zener_Small
- PT0: symbol Connector:Conn_01x03_Female -> UCIRP-KiCAD-Lib:Conn_01x03_Female
- R10, R11, R12: symbol Device:R_Small_US -> UCIRP-KiCAD-Lib:R_Small_US
- U8: value OPA357 -> ~; symbol ECU:OPA357 -> UCIRP-KiCAD-Lib:OPA357

Commit message: fix
Parts:
- PT0: Manufacturer Generic -> (none); Part # Generic 3x5.08 Screw Terminal -> (none)
- R10: Part # Generic 1K 0402 Resistor -> Generic 1K 1% 0402 Resistor
- R11: Part # Generic 4.7K 0402 Resistor -> Generic 4.7K 1% 0402 Resistor
- R12: value 4.7K -> 10K; Part # Generic 4.7K 0402 Resistor -> Generic 10K 1% 0402 Resistor
Changed lines of the file:
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@@
       (effects (font (size 1.27 1.27)) hide)
     )
-    (property "Manufacturer" "Generic" (at 71.12 54.61 0)
-      (effects (font (size 1.27 1.27)) hide)
-    )
-    (property "Part #" "Generic 3x5.08 Screw Terminal" (at 71.12 54.61 0)
+    (property "Manufacturer" "~" (at 71.12 54.61 0)
+      (effects (font (size 1.27 1.27)) hide)
+    )
+    (property "Part #" "~" (at 71.12 54.61 0)
       (effects (font (size 1.27 1.27)) hide)
     )
@@
       (effects (font (size 1.27 1.27)) hide)
     )
-    (property "Part #" "Generic 1K 0402 Resistor" (at 81.28 54.61 0)
+    (property "Part #" "Generic 1K 1% 0402 Resistor" (at 81.28 54.61 0)
       (effects (font (size 1.27 1.27)) hide)
     )
@@
       (effects (font (size 1.27 1.27)) hide)
     )
-    (property "Part #" "Generic 4.7K 0402 Resistor" (at 120.65 60.96 0)
+    (property "Part #" "Generic 4.7K 1% 0402 Resistor" (at 120.65 60.96 0)
       (effects (font (size 1.27 1.27)) hide)
     )
@@
       (effects (font (size 1.27 1.27)) (justify left))
     )
-    (property "Value" "4.7K" (at 123.19 72.39 0)
+    (property "Value" "10K" (at 123.19 72.39 0)
       (effects (font (size 1.27 1.27)) (justify left))
     )
@@
       (effects (font (size 1.27 1.27)) hide)
     )
-    (property "Part #" "Generic 4.7K 0402 Resistor" (at 120.65 71.12 0)
-      (effects (font (size 1.27 1.27)) hide)
-    )
+    (property "Part #" "Generic 10K 1% 0402 Resistor" (at 120.65 71.12 0)
+      (effects (font (size 1.27 1.27)) hide)
+    )

Commit message: finished pcb design of gse 1.0
Parts:
- D?: renamed from D3; value 5V -> 5.1V
- R?: renamed from R11; value 4.7K -> 5K; Part # Generic 4.7K 1% 0402 Resistor -> Generic 5K 1% 0402 Resistor
- renumbered C30 to C?, PT0 to PT?, R10 to R?, R12 to R?, U8 to U?
