File: ignition.kicad_sch (KiCad schematic)
At the start: 8 parts, among them J3 E-MATCH_IGNITION1, Q1 Q_NMOS_GSD, Q2 Q_NMOS_GSD

Commit message: fix
Parts:
- added R3, R4: 10K, Resistor_SMD:R_0402_1005Metric, symbol Device:R_Small_US
- J3: value E-MATCH_IGNITION1 -> E-MATCH; Manufacturer Generic -> (none); Part # Generic 2x5.08 Screw Terminal -> (none)
- Q1, Q2: value Q_NMOS_GSD -> ~; footprint Package_TO_SOT_SMD:TSOT-23 -> Package_TO_SOT_SMD:SOT-23-3; Manufacturer nexperia -> Diodes; Part # PMV30UN2 -> DMG3402L
- R3, R4: value 1K -> 10K; Part # Generic 1K 0402 Resistor -> Generic 10K 1% 0402 Resistor
- R5: Part # Generic 10K 0402 Resistor -> Generic 10K 1% 0402 Resistor
- R5: Part # Generic 100 0402 Resistor -> Generic 100 1% 0402 Resistor
Connections:
- net GND: now also R3.2
- net at J3.2 (Pin_2), Q2.3 (D), R4.1: now also R4.1; no longer Q1.1 (G)
- new net: Q1.1 (G), R3.1, R4.2
Other:
- moved on the sheet: Q1, R3

Commit message: finished pcb design of gse 1.0
Parts:
- removed R4: 10K, Resistor_SMD:R_0402_1005Metric, symbol Device:R_Small_US
- Q?: renamed from Q2; value ~ -> 30V 4A
- Q?: renamed from Q1; value ~ -> 30V 4A
- R?: renamed from R4; value 10K -> 33K; Part # Generic 10K 1% 0402 Resistor -> Generic 33K 1% 0402 Resistor
- R?: renamed from R5; Part # Generic 100 1% 0402 Resistor -> Generic 15K 1% 0402 Resistor
- renumbered C8 to C?, J3 to J?, R3 to R?, R5 to R?
Other:
- moved on the sheet: Q?, R?

Commit message: fixed resistor values
Parts:
- R?: Part # Generic 15K 1% 0402 Resistor -> Generic 100 1% 0402 Resistor
Changed lines of the file:
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@@
       (effects (font (size 1.27 1.27)) hide)
     )
-    (property "Part #" "Generic 15K 1% 0402 Resistor" (at 142.875 100.33 0)
+    (property "Part #" "Generic 100 1% 0402 Resistor" (at 142.875 100.33 0)
       (effects (font (size 1.27 1.27)) hide)
     )
