File: rocket2-gse-hardware.kicad_sch (KiCad schematic)
At the start: 64 parts, among them J1 ARMING_PLUG, J1 USB_C Connector, J8 ALARM, J8 PWR, Y1 16MHz

Commit message: finished pcb design of gse 1.0
Parts:
- D10: renamed from D9; footprint (none) -> Diode_SMD:D_SMA; Manufacturer Vishay -> Micro Commercial Co; Part # V8PAM10HM3/I -> SL310A-TP
- D11: renamed from D10; footprint (none) -> Diode_SMD:D_SMA; Manufacturer Vishay -> Micro Commercial Co; Part # V8PAM10HM3/I -> SL310A-TP
- D12: renamed from D11; footprint (none) -> Diode_SMD:D_SMA; Manufacturer Vishay -> Micro Commercial Co; Part # V8PAM10HM3/I -> SL310A-TP
- D13: renamed from D12; footprint (none) -> Diode_SMD:D_SMA; Manufacturer Vishay -> Micro Commercial Co; Part # V8PAM10HM3/I -> SL310A-TP
- D6: renamed from D5; footprint (none) -> Diode_SMD:D_SMA; Manufacturer Vishay -> Micro Commercial Co; Part # V8PAM10HM3/I -> SL310A-TP
- D7: renamed from D6; footprint (none) -> Diode_SMD:D_SMA; Manufacturer Vishay -> Micro Commercial Co; Part # V8PAM10HM3/I -> SL310A-TP
- D8: renamed from D7; footprint (none) -> Diode_SMD:D_SMA; Manufacturer Vishay -> Micro Commercial Co; Part # V8PAM10HM3/I -> SL310A-TP
- D9: renamed from D8; footprint (none) -> Diode_SMD:D_SMA; Manufacturer Vishay -> Micro Commercial Co; Part # V8PAM10HM3/I -> SL310A-TP
- F1: footprint (none) -> Fuse:Fuseholder_Blade_Mini_Keystone_3568
- J? (x2): renamed from J8; footprint TerminalBlock:TerminalBlock_bornier-2_P5.08mm -> Connector_BarrelJack:BarrelJack_Horizontal
- Q?: renamed from Q2; value ~ -> 30V 4A
- R13: renamed from R12; value 100k -> 100K; Part # Generic 68K 1% 0402 Resistor -> Generic 100K 1% 0402 Resistor
- R14: renamed from R13; value 15k -> 15K; Part # Generic 10K 1% 0402 Resistor -> Generic 15K 1% 0402 Resistor
- R17: renamed from R16; value 100k -> 100K; Part # Generic 68K 1% 0402 Resistor -> Generic 100K 1% 0402 Resistor
- R18: renamed from R17; value 15k -> 15K; Part # Generic 10K 1% 0402 Resistor -> Generic 15K 1% 0402 Resistor
- R?: renamed from R1; Part # Generic 68K 1% 0402 Resistor -> Generic 100K 1% 0402 Resistor
- R?: renamed from R30; Part # Generic 470 1% 0402 Resistor -> Generic 100K 1% 0402 Resistor
- R?: renamed from R2; Part # Generic 10K 1% 0402 Resistor -> Generic 15K 1% 0402 Resistor
- R?: renamed from R13; Part # Generic 100 1% 0402 Resistor -> Generic 15K 1% 0402 Resistor
- renumbered C3 to C?, C2 to C?, C5 to C?, C39 to C?, C4 to C?, C9 to C?, C6 to C?, C38 to C?, D11 to D?, D10 to D?, D9 to D?, J1 to J?, J8 to J?, R28 to R?, R32 to R?, R13 to R?, R31 to R?, R14 to R?, R29 to R?, TP3 to TP?, TP2 to TP?, TP1 to TP?, Y1 to Y?
Connections:
- net IGNITION2_CONT is gone; now on net IGNITION1_CONT: U1.38 (PC7)
- net IGNITION2_OUTPUT is gone; now on net IGNITION1_OUTPUT: U1.36 (PB15)
- net PWR_READ2 is gone; now on net PWR_READ1: R17.2, R18.1, U1.27 (PB1)
- net +24V: now also TP?.1; no longer TP?.1
- net +3.3V: now also TP?.1; no longer TP?.1
- net IGNITION0_CONT: now also U1.39 (PC8)
- net IGNITION0_OUTPUT: now also U1.37 (PC6)
- net IGNITION1_CONT: no longer U1.39 (PC8)
- net IGNITION1_OUTPUT: no longer U1.37 (PC6)
- net PWR_READ1: no longer R13.2, R14.1, U1.26 (PB0)
- net ALARM_EN0 renamed ALARM_EN
- net PWR1 renamed PWR0
- net PWR0: now also TP?.1; no longer TP?.1
- new net PWR_READ0: R13.2, R14.1, U1.26 (PB0)
Other:
- moved on the sheet: D?, R?, TP?

Commit message: fixed resistor values
Parts:
- R?: Part # Generic 100K 1% 0402 Resistor -> Generic 470 1% 0402 Resistor
- R?: Part # Generic 15K 1% 0402 Resistor -> Generic 100 1% 0402 Resistor
Changed lines of the file:
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@@
       (effects (font (size 1.27 1.27)) hide)
     )
-    (property "Part #" "Generic 100K 1% 0402 Resistor" (at 187.96 179.705 0)
+    (property "Part #" "Generic 470 1% 0402 Resistor" (at 187.96 179.705 0)
       (effects (font (size 1.27 1.27)) hide)
     )
@@
       (effects (font (size 1.27 1.27)) hide)
     )
-    (property "Part #" "Generic 15K 1% 0402 Resistor" (at 267.97 229.87 0)
-      (effects (font (size 1.27 1.27)) hide)
-    )
+    (property "Part #" "Generic 100 1% 0402 Resistor" (at 267.97 229.87 0)
+      (effects (font (size 1.27 1.27)) hide)
+    )
