File: solenoids.kicad_sch (KiCad schematic)
At the start: 9 parts, among them J2 Solenoid, U5 OPA357

Commit message: fixed resistor values
Parts:
- R13: Part # Generic 1K 0402 Resistor -> Generic 1 0402 Resistor
Changed lines of the file:
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@@
       (effects (font (size 1.27 1.27)) hide)
     )
-    (property "Part #" "Generic 1K 0402 Resistor" (at 80.01 62.23 0)
+    (property "Part #" "Generic 1 0402 Resistor" (at 80.01 62.23 0)
       (effects (font (size 1.27 1.27)) hide)
     )

Commit message: added full schematic and outdated pcb
Parts:
- removed J2: Solenoid, TerminalBlock:TerminalBlock_bornier-2_P5.08mm, symbol Connector:Conn_01x02_Female
- added PT0: Solenoid, TerminalBlock:TerminalBlock_bornier-3_P5.08mm, symbol UCIRP-KiCAD-Lib:Conn_01x03_Female
- added R13: 100, Resistor_SMD:R_0402_1005Metric, symbol UCIRP-KiCAD-Lib:R_Small_US
- C34: symbol Device:C_Small -> UCIRP-KiCAD-Lib:C_Small
- D2: value ~ -> 1.0A; symbol Device:D_Schottky_Small -> UCIRP-KiCAD-Lib:D_Schottky_Small
- D4: footprint Diode_SMD:D_MiniMELF -> Diode_SMD:D_SOD-123; symbol Device:D_Zener_Small -> UCIRP-KiCAD-Lib:D_Zener_Small
- Q2: value ~ -> n-MOSFET; footprint Package_TO_SOT_THT:TO-220-3_Vertical -> Package_TO_SOT_SMD:SOT-23-3; symbol Device:Q_NMOS_GDS -> UCIRP-KiCAD-Lib:Q_NMOS_GDS
- R13: value 4.7K -> 10K; symbol Device:R_Small_US -> UCIRP-KiCAD-Lib:R_Small_US; Part # Generic 1K 0402 Resistor -> Generic 10K 0402 Resistor
- R13: footprint Resistor_SMD:R_0402_1005Metric -> Resistor_SMD:R_1206_3216Metric; symbol Device:R_Small_US -> UCIRP-KiCAD-Lib:R_Small_US; Part # Generic 1 0402 Resistor -> Generic 1 1206 Resistor
- R13: symbol Device:R_Small_US -> UCIRP-KiCAD-Lib:R_Small_US
- U5: value OPA357 -> ~; symbol ECU:OPA357 -> UCIRP-KiCAD-Lib:OPA357
Connections:
- net +24V: now also D2.2 (A), PT0.1 (Pin_1); no longer D2.1 (K)
- net GND: now also PT0.3 (Pin_3)
- net S_EN: now also R13.1; no longer Q2.1 (G)
- net at Q2.2 (D): now also D2.1 (K), PT0.2 (Pin_2); no longer D2.2 (A)
- new net: Q2.1 (G), R13.2
Other:
- moved on the sheet: D2, R13

Commit message: final polished schematic b4 daniel fixes nmosfet and ignition circuit
Parts:
- R13: Part # Generic 10K 0402 Resistor -> Generic 100 0402 Resistor
Other:
- moved on the sheet: C34, D2, D4, PT0, Q2, R13, U5

Commit message: fix
Parts:
- PT0: Manufacturer Generic -> (none); Part # Generic 3x5.08 Screw Terminal -> (none)
- Q2: value n-MOSFET -> ~; symbol UCIRP-KiCAD-Lib:Q_NMOS_GDS -> Device:Q_NMOS_GSD
- R13: Part # Generic 100 0402 Resistor -> Generic 100 1% 0402 Resistor
- R13: Part # Generic 10K 0402 Resistor -> Generic 10K 1% 0402 Resistor
- R13: Part # Generic 1 1206 Resistor -> Generic 1 1% 1206 Resistor
- R13: Part # Generic 1K 0402 Resistor -> Generic 1K 1% 0402 Resistor
Connections:
- net at D2.1 (K), PT0.2 (Pin_2): now also Q2.3 (D); no longer Q2.2 (D)
- net at R13.1, R13.1: now also Q2.2 (S); no longer Q2.3 (S)
Changed lines of the file:
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@@
       (effects (font (size 1.27 1.27)) hide)
     )
-    (property "Part #" "Generic 100 0402 Resistor" (at 74.93 52.07 0)
+    (property "Part #" "Generic 100 1% 0402 Resistor" (at 74.93 52.07 0)
       (effects (font (size 1.27 1.27)) hide)
     )
@@
       (effects (font (size 1.27 1.27)) hide)
     )
-    (property "Part #" "Generic 10K 0402 Resistor" (at 65.405 56.515 0)
+    (property "Part #" "Generic 10K 1% 0402 Resistor" (at 65.405 56.515 0)
       (effects (font (size 1.27 1.27)) hide)
     )
@@
     )
   )
-  (symbol (lib_id "UCIRP-KiCAD-Lib:Q_NMOS_GDS") (at 87.63 52.07 0) (unit 1)
+  (symbol (lib_id "Device:Q_NMOS_GSD") (at 87.63 52.07 0) (unit 1)
     (in_bom yes) (on_board yes) (dnp no)
     (property "Reference" "Q2" (at 92.71 52.07 0)
       (effects (font (size 1.27 1.27)) (justify left))
     )
-    (property "Value" "n-MOSFET" (at 92.71 53.34 0)
+    (property "Value" "~" (at 92.71 53.34 0)
       (effects (font (size 1.27 1.27)) (justify left))
     )
@@
       (effects (font (size 1.27 1.27)) hide)
     )
-    (property "Part #" "Generic 1 1206 Resistor" (at 90.17 62.23 0)
+    (property "Part #" "Generic 1 1% 1206 Resistor" (at 90.17 62.23 0)
       (effects (font (size 1.27 1.27)) hide)
     )
@@
       (effects (font (size 1.27 1.27)) hide)
     )
-    (property "Manufacturer" "Generic" (at 82.55 40.64 0)
-      (effects (font (size 1.27 1.27)) hide)
-    )
-    (property "Part #" "Generic 3x5.08 Screw Terminal" (at 82.55 40.64 0)
+    (property "Manufacturer" "~" (at 82.55 40.64 0)
+      (effects (font (size 1.27 1.27)) hide)
+    )
+    (property "Part #" "~" (at 82.55 40.64 0)
       (effects (font (size 1.27 1.27)) hide)
     )
@@
       (effects (font (size 1.27 1.27)) hide)
     )
-    (property "Part #" "Generic 1K 0402 Resistor" (at 96.52 58.42 0)
-      (effects (font (size 1.27 1.27)) hide)
-    )
+    (property "Part #" "Generic 1K 1% 0402 Resistor" (at 96.52 58.42 0)
+      (effects (font (size 1.27 1.27)) hide)
+    )

Commit message: Added in dual power, fuse, status led, and comments
Other:
- moved on the sheet: D2, R13

Commit message: finished pcb design of gse 1.0
Parts:
- Q?: renamed from Q2; value ~ -> 30V 4A
- R?: renamed from R13; Part # Generic 100 1% 0402 Resistor -> Generic 15K 1% 0402 Resistor
- renumbered C34 to C?, D4 to D?, D2 to D?, PT0 to PT?, R13 to R?, U5 to U?
Connections:
- net +24V: now also D?.1 (K); no longer D?.2 (A)
- net at PT?.2 (Pin_2), Q?.3 (D): now also D?.2 (A); no longer D?.1 (K)

Commit message: fixed resistor values
Parts:
- R?: Part # Generic 15K 1% 0402 Resistor -> Generic 100 1% 0402 Resistor
Changed lines of the file:
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@@
       (effects (font (size 1.27 1.27)) hide)
     )
-    (property "Part #" "Generic 15K 1% 0402 Resistor" (at 74.93 52.07 0)
+    (property "Part #" "Generic 100 1% 0402 Resistor" (at 74.93 52.07 0)
       (effects (font (size 1.27 1.27)) hide)
     )
