File: rocket2-gse-hardware.kicad_pcb (KiCad board)
At the start: 4 copper layers, 173 x 147 mm, 243 parts, among them J1 ARMING_PLUG, J2 ALARM, J3 USB_C Connector, J4 PWR, J5 PWR, J6 E-MATCH, J7 E-MATCH, Q1 30V 4A, Q10 30V 4A, Q11 30V 4A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

Commit message: Fix planes
Parts:
- moved U3 88.3 mm to (100.0, 157.0)
- moved U4 42.5 mm to (141.9, 133.9), turned to 180 degrees
- moved D6 28.0 mm to (116.7, 43.0), turned to 90 degrees
- moved R17 26.7 mm to (137.7, 41.5), turned to -90 degrees
- moved F1 23.3 mm to (93.0, 24.3)
- moved R18 23.2 mm to (137.7, 44.0), turned to -90 degrees
- moved D7 21.5 mm to (121.7, 43.0), turned to 90 degrees
- moved D10 20.3 mm to (140.7, 43.0), turned to 90 degrees
- moved R13 19.0 mm to (134.7, 41.5), turned to -90 degrees
- moved R14 16.0 mm to (134.7, 43.8), turned to -90 degrees
- moved D8 15.5 mm to (126.7, 43.0), turned to 90 degrees
- moved J4 13.3 mm to (128.7, 34.5)
- moved J5 13.3 mm to (143.7, 34.5)
- moved D11 13.3 mm to (145.7, 43.0), turned to 90 degrees
- moved D9 10.8 mm to (131.7, 43.0), turned to 90 degrees
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Routing:
- net +24V: track 759.8 -> 0.00 mm, vias 1 -> 0
- net TC_SPI1_SO: track 213.4 -> 0.00 mm, vias 2 -> 0
- net TC_SPI1_SCK: track 205.0 -> 0.00 mm, vias 2 -> 0
- net +3.3V: track 159.1 -> 0.00 mm, vias 26 -> 0
- net PWR0: track 148.4 -> 0.00 mm, vias 2 -> 0
- net +5V: track 109.0 -> 0.00 mm, vias 6 -> 0
- net ALARM_EN: track 105.3 -> 0.00 mm, vias 2 -> 0
- net IGNITION1_CONT: track 96.9 -> 0.00 mm, vias 2 -> 0
- net ARM_CONT: track 91.0 -> 0.00 mm, vias 2 -> 0
- net USB_VBUS: track 87.9 -> 0.00 mm, vias 3 -> 0
- net IGNITION0_CONT: track 84.2 -> 0.00 mm, vias 2 -> 0
- net S_EN8: track 83.6 -> 0.00 mm, vias 2 -> 0
- net nCS_5: track 80.0 -> 0.00 mm, vias 2 -> 0
- net S_FB8: track 78.8 -> 0.00 mm
- net S_EN6: track 78.4 -> 0.00 mm, vias 2 -> 0
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- added copper zone on F.Cu, net +24V
- added copper zone on In2.Cu, net +24V
- added copper zone on F.Cu, net Net-(D10-A)
- added copper zone on F.Cu, net Net-(D6-A)
- added copper zone on F.Cu, net PWR0
Other:
- outline, holes or cut-outs redrawn
